File: tusb211.sch (EAGLE design)
At the start: 11 parts, among them U1 Value

Commit message: Got rid of PCB USB, added led, added spot for EQ resistor, fixed wiring
Parts:
- removed BOARDTOPI: USBPCB, USBPCB:USBPCB
- added D2: GREEN, SparkFun-LED:LED-GREEN0603
- added R2, VARIABLER: 120, rcl:R-US_R0805
- added U$1: TYPEAUSB, TYPEAUSBSMDMALE:TYPEAUSB
- renumbered USBSMD to U$2
Connections:
- removed net EQ: U1.EQ
- new net N$5: U1.EQ, VARIABLER.2
- new net N$6: R2.2, U1.ENA_HS
- new net N$7: D2.A, R2.1
- net 3.3V: now also VOLTAGEREGULATOR.VIN+
- net GND: now also D2.C, U$1.GND, VARIABLER.1; no longer BOARDTOPI.GND
- net M: now also U$1.D-; no longer BOARDTOPI.D-
- net P: now also U$1.D+; no longer BOARDTOPI.D+
- net VIN: now also U$1.VCC; no longer BOARDTOPI.VCC, VOLTAGEREGULATOR.VIN+
Other:
- moved on the sheet: D1, R1
